File: hardware/1w-If.kicad_sch (KiCad schematic)
At the start: 50 parts, among them U1 WT32-ETH01, U2 TCA9548APWR, U3 DS2484R, U4 DS2484R, U5 DS2484R, U6 DS2484R, X1 PowerSupply, X2 Debug Terminal, X3 Ext LED Terminal, X4 1-Wire Ch1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

Commit message: PCB v1.1 (#9)
- Add missing polarity of tantal capacities C1-C4.
- Too bright LEDs: R1-R4 changed to 1kOhm
- Swapped ext. LED connector silk layer description
Parts:
- added D3: LED Power ext. 20mA, LED_SMD:LED_0805_2012Metric_Pad1.15x1.40mm_HandSolder, symbol Device:LED
- added D4: LED Status ext. 20mA, LED_SMD:LED_0805_2012Metric_Pad1.15x1.40mm_HandSolder, symbol Device:LED
- C1, C2, C3, C4: symbol Device:C -> Device:C_Polarized
- D1: value LED Power -> LED Power 5mA
- D2: value LED Status -> LED Status 5mA
- R1, R2, R3, R4: value 100 -> 1k
Connections:
- net +3.3V: now also C4.1; no longer C4.2
- net +5V: now also C1.1, C2.1; no longer C1.2, C2.2
- net GND: now also C1.2, C2.2, C3.2, C4.2, D3.1 (K); no longer C1.1, C2.1, C3.1, C4.1
- net LED_Status-: now also D4.1 (K)
- net WT32_ETH01_EN: now also C3.1; no longer C3.2
- net at R3.1, X3.1 (Pin_1): now also D4.2 (A)
- net at R1.1, X3.3 (Pin_3): now also D3.2 (A)
Other:
- moved on the sheet: D1, D2, H1, H2, H3, H4, H5, H6, R1, R2, R3, R4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
