File: hardware/1w-If.kicad_pcb (KiCad board)
At the start: 2 copper layers, 68 x 85 mm, 50 parts, among them U1 WT32-ETH01, U2 TCA9548APWR, U3 DS2484R, U4 DS2484R, U5 DS2484R, U6 DS2484R, X1 PowerSupply, X2 Debug Terminal, X3 Ext LED Terminal, X4 1-Wire Ch1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

Commit message: PCB v1.1 (#9)
- Add missing polarity of tantal capacities C1-C4.
- Too bright LEDs: R1-R4 changed to 1kOhm
- Swapped ext. LED connector silk layer description
Parts:
- D1: value LED Power -> LED Power 5mA
- D2: value LED Status -> LED Status 5mA
- R1, R2, R3, R4: value 100 -> 1k
- moved C6 71.2 mm to (109.0, 113.8)
- moved C7 71.2 mm to (100.6, 113.8)
- moved C8 71.2 mm to (92.5, 113.8)
- moved C9 71.2 mm to (84.0, 113.8)
- moved U2 70.7 mm to (101.7, 138.4)
- moved R15 70.7 mm to (92.5, 122.5)
- moved R16 70.7 mm to (94.5, 122.5)
- moved R17 70.7 mm to (90.5, 122.5)
- moved U5 70.7 mm to (92.5, 117.4)
- moved X1 70.7 mm to (83.4, 170.7)
- moved X2 70.7 mm to (93.9, 170.7)
- moved C1 70.7 mm to (83.4, 152.8), turned to 180 degrees
- moved C2 70.7 mm to (83.4, 150.5), turned to 180 degrees
- moved C3 70.7 mm to (131.0, 128.5), turned to -90 degrees
- moved C4 70.7 mm to (131.0, 149.0), turned to 90 degrees
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Connections:
- C1 pad 1: GND -> +5V
- C1 pad 2: +5V -> GND
- C2 pad 1: GND -> +5V
- C2 pad 2: +5V -> GND
- C3 pad 1: GND -> /WT32_ETH01_EN
- C3 pad 2: /WT32_ETH01_EN -> GND
- C4 pad 1: GND -> +3.3V
- C4 pad 2: +3.3V -> GND
Routing:
- net +5V: track 332.0 -> 328.7 mm
- net GND: track 415.8 -> 414.7 mm
- net /OW_Ch2: track 32.9 -> 32.3 mm
Other:
- board text added: "v 1.1"
- board text removed: "v 1.0"
